Commit message: Added collision geometries

File: tb4_lss_arm/lss_arm_description/urdf/lss_arm/lss_arm.urdf.xacro (robot description, xacro)
@@ -15,14 +15,14 @@
             <origin xyz="0 0 0" rpy="0 0 0" />
             <geometry>
-                <mesh filename="package://lss_arm_description/meshes/link_0.STL" />
-            </geometry>
-            <material name="">
-                <color rgba="0.3 0.3 0.3 1" />
-            </material>
-        </visual>
-        <collision>
-            <origin xyz="0 0 0" rpy="0 0 0" />
-            <geometry>
-                <mesh filename="package://lss_arm_description/meshes/link_0.STL" />
+                <mesh filename="package://lss_arm_description/meshes/visual/link_0.STL" />
+            </geometry>
+            <material name="">
+                <color rgba="0.3 0.3 0.3 1" />
+            </material>
+        </visual>
+        <collision>
+            <origin xyz="0 0 0" rpy="0 0 0" />
+            <geometry>
+                <mesh filename="package://lss_arm_description/meshes/collision/link_0.STL" />
             </geometry>
         </collision>
@@ -41,14 +41,14 @@
             <origin xyz="0 0 0" rpy="0 0 0" />
             <geometry>
-                <mesh filename="package://lss_arm_description/meshes/link_1.STL" />
-            </geometry>
-            <material name="">
-                <color rgba="0.3 0.3 0.3 1" />
-            </material>
-        </visual>
-        <collision>
-            <origin xyz="0 0 0" rpy="0 0 0" />
-            <geometry>
-                <mesh filename="package://lss_arm_description/meshes/link_1.STL" />
+                <mesh filename="package://lss_arm_description/meshes/visual/link_1.STL" />
+            </geometry>
+            <material name="">
+                <color rgba="0.3 0.3 0.3 1" />
+            </material>
+        </visual>
+        <collision>
+            <origin xyz="0 0 0" rpy="0 0 0" />
+            <geometry>
+                <mesh filename="package://lss_arm_description/meshes/collision/link_1.STL" />
             </geometry>
         </collision>
@@ -70,14 +70,14 @@
             <origin xyz="0 0 0" rpy="0 0 0" />
             <geometry>
-                <mesh filename="package://lss_arm_description/meshes/link_2.STL" />
-            </geometry>
-            <material name="">
-                <color rgba="0.3 0.3 0.3 1" />
-            </material>
-        </visual>
-        <collision>
-            <origin xyz="0 0 0" rpy="0 0 0" />
-            <geometry>
-                <mesh filename="package://lss_arm_description/meshes/link_2.STL" />
+                <mesh filename="package://lss_arm_description/meshes/visual/link_2.STL" />
+            </geometry>
+            <material name="">
+                <color rgba="0.3 0.3 0.3 1" />
+            </material>
+        </visual>
+        <collision>
+            <origin xyz="0 0 0" rpy="0 0 0" />
+            <geometry>
+                <mesh filename="package://lss_arm_description/meshes/collision/link_2.STL" />
             </geometry>
         </collision>
@@ -99,14 +99,14 @@
             <origin xyz="0 0 0" rpy="0 0 0" />
             <geometry>
-                <mesh filename="package://lss_arm_description/meshes/link_3.STL" />
-            </geometry>
-            <material name="">
-                <color rgba="0.3 0.3 0.3 1" />
-            </material>
-        </visual>
-        <collision>
-            <origin xyz="0 0 0" rpy="0 0 0" />
-            <geometry>
-                <mesh filename="package://lss_arm_description/meshes/link_3.STL" />
+                <mesh filename="package://lss_arm_description/meshes/visual/link_3.STL" />
+            </geometry>
+            <material name="">
+                <color rgba="0.3 0.3 0.3 1" />
+            </material>
+        </visual>
+        <collision>
+            <origin xyz="0 0 0" rpy="0 0 0" />
+            <geometry>
+                <mesh filename="package://lss_arm_description/meshes/collision/link_3.STL" />
             </geometry>
         </collision>
@@ -128,14 +128,14 @@
             <origin xyz="0 0 0" rpy="0 0 0" />
             <geometry>
-                <mesh filename="package://lss_arm_description/meshes/link_4.STL" />
-            </geometry>
-            <material name="">
-                <color rgba="0.3 0.3 0.3 1" />
-            </material>
-        </visual>
-        <collision>
-            <origin xyz="0 0 0" rpy="0 0 0" />
-            <geometry>
-                <mesh filename="package://lss_arm_description/meshes/link_4.STL" />
+                <mesh filename="package://lss_arm_description/meshes/visual/link_4.STL" />
+            </geometry>
+            <material name="">
+                <color rgba="0.3 0.3 0.3 1" />
+            </material>
+        </visual>
+        <collision>
+            <origin xyz="0 0 0" rpy="0 0 0" />
+            <geometry>
+                <mesh filename="package://lss_arm_description/meshes/collision/link_4.STL" />
             </geometry>
         </collision>
@@ -157,14 +157,14 @@
             <origin xyz="0 0 0" rpy="0 0 0" />
             <geometry>
-                <mesh filename="package://lss_arm_description/meshes/end_effector_r.STL" />
-            </geometry>
-            <material name="">
-                <color rgba="0.3 0.3 0.3 1" />
-            </material>
-        </visual>
-        <collision>
-            <origin xyz="0 0 0" rpy="0 0 0" />
-            <geometry>
-                <mesh filename="package://lss_arm_description/meshes/end_effector_r.STL" />
+                <mesh filename="package://lss_arm_description/meshes/visual/end_effector_r.STL" />
+            </geometry>
+            <material name="">
+                <color rgba="0.3 0.3 0.3 1" />
+            </material>
+        </visual>
+        <collision>
+            <origin xyz="0 0 0" rpy="0 0 0" />
+            <geometry>
+                <mesh filename="package://lss_arm_description/meshes/collision/end_effector_r.STL" />
             </geometry>
         </collision>
@@ -186,14 +186,14 @@
             <origin xyz="0 0 0" rpy="0 0 0" />
             <geometry>
-                <mesh filename="package://lss_arm_description/meshes/end_effector_l.STL" />
-            </geometry>
-            <material name="">
-                <color rgba="0.3 0.3 0.3 1" />
-            </material>
-        </visual>
-        <collision>
-            <origin xyz="0 0 0" rpy="0 0 0" />
-            <geometry>
-                <mesh filename="package://lss_arm_description/meshes/end_effector_l.STL" />
+                <mesh filename="package://lss_arm_description/meshes/visual/end_effector_l.STL" />
+            </geometry>
+            <material name="">
+                <color rgba="0.3 0.3 0.3 1" />
+            </material>
+        </visual>
+        <collision>
+            <origin xyz="0 0 0" rpy="0 0 0" />
+            <geometry>
+                <mesh filename="package://lss_arm_description/meshes/collision/end_effector_l.STL" />
             </geometry>
         </collision>

File: tb4_lss_arm/lss_arm_description/urdf/tb4_lss_arm/tb4_lss_arm.urdf.xacro (robot description, xacro)
@@ -16,14 +16,14 @@
             <origin xyz="0 0 0" rpy="0 0 0" />
             <geometry>
-                <mesh filename="package://lss_arm_description/meshes/link_0.STL" />
-            </geometry>
-            <material name="">
-                <color rgba="0.3 0.3 0.3 1" />
-            </material>
-        </visual>
-        <collision>
-            <origin xyz="0 0 0" rpy="0 0 0" />
-            <geometry>
-                <mesh filename="package://lss_arm_description/meshes/link_0.STL" />
+                <mesh filename="package://lss_arm_description/meshes/visual/link_0.STL" />
+            </geometry>
+            <material name="">
+                <color rgba="0.3 0.3 0.3 1" />
+            </material>
+        </visual>
+        <collision>
+            <origin xyz="0 0 0" rpy="0 0 0" />
+            <geometry>
+                <mesh filename="package://lss_arm_description/meshes/collision/link_0.STL" />
             </geometry>
         </collision>
@@ -43,14 +43,14 @@
             <origin xyz="0 0 0" rpy="0 0 0" />
             <geometry>
-                <mesh filename="package://lss_arm_description/meshes/link_1.STL" />
-            </geometry>
-            <material name="">
-                <color rgba="0.3 0.3 0.3 1" />
-            </material>
-        </visual>
-        <collision>
-            <origin xyz="0 0 0" rpy="0 0 0" />
-            <geometry>
-                <mesh filename="package://lss_arm_description/meshes/link_1.STL" />
+                <mesh filename="package://lss_arm_description/meshes/visual/link_1.STL" />
+            </geometry>
+            <material name="">
+                <color rgba="0.3 0.3 0.3 1" />
+            </material>
+        </visual>
+        <collision>
+            <origin xyz="0 0 0" rpy="0 0 0" />
+            <geometry>
+                <mesh filename="package://lss_arm_description/meshes/collision/link_1.STL" />
             </geometry>
         </collision>
@@ -72,14 +72,14 @@
             <origin xyz="0 0 0" rpy="0 0 0" />
             <geometry>
-                <mesh filename="package://lss_arm_description/meshes/link_2.STL" />
-            </geometry>
-            <material name="">
-                <color rgba="0.3 0.3 0.3 1" />
-            </material>
-        </visual>
-        <collision>
-            <origin xyz="0 0 0" rpy="0 0 0" />
-            <geometry>
-                <mesh filename="package://lss_arm_description/meshes/link_2.STL" />
+                <mesh filename="package://lss_arm_description/meshes/visual/link_2.STL" />
+            </geometry>
+            <material name="">
+                <color rgba="0.3 0.3 0.3 1" />
+            </material>
+        </visual>
+        <collision>
+            <origin xyz="0 0 0" rpy="0 0 0" />
+            <geometry>
+                <mesh filename="package://lss_arm_description/meshes/collision/link_2.STL" />
             </geometry>
         </collision>
@@ -101,14 +101,14 @@
             <origin xyz="0 0 0" rpy="0 0 0" />
             <geometry>
-                <mesh filename="package://lss_arm_description/meshes/link_3.STL" />
-            </geometry>
-            <material name="">
-                <color rgba="0.3 0.3 0.3 1" />
-            </material>
-        </visual>
-        <collision>
-            <origin xyz="0 0 0" rpy="0 0 0" />
-            <geometry>
-                <mesh filename="package://lss_arm_description/meshes/link_3.STL" />
+                <mesh filename="package://lss_arm_description/meshes/visual/link_3.STL" />
+            </geometry>
+            <material name="">
+                <color rgba="0.3 0.3 0.3 1" />
+            </material>
+        </visual>
+        <collision>
+            <origin xyz="0 0 0" rpy="0 0 0" />
+            <geometry>
+                <mesh filename="package://lss_arm_description/meshes/collision/link_3.STL" />
             </geometry>
         </collision>
@@ -130,14 +130,14 @@
             <origin xyz="0 0 0" rpy="0 0 0" />
             <geometry>
-                <mesh filename="package://lss_arm_description/meshes/link_4.STL" />
-            </geometry>
-            <material name="">
-                <color rgba="0.3 0.3 0.3 1" />
-            </material>
-        </visual>
-        <collision>
-            <origin xyz="0 0 0" rpy="0 0 0" />
-            <geometry>
-                <mesh filename="package://lss_arm_description/meshes/link_4.STL" />
+                <mesh filename="package://lss_arm_description/meshes/visual/link_4.STL" />
+            </geometry>
+            <material name="">
+                <color rgba="0.3 0.3 0.3 1" />
+            </material>
+        </visual>
+        <collision>
+            <origin xyz="0 0 0" rpy="0 0 0" />
+            <geometry>
+                <mesh filename="package://lss_arm_description/meshes/collision/link_4.STL" />
             </geometry>
         </collision>
@@ -159,14 +159,14 @@
             <origin xyz="0 0 0" rpy="0 0 0" />
             <geometry>
-                <mesh filename="package://lss_arm_description/meshes/end_effector_r.STL" />
-            </geometry>
-            <material name="">
-                <color rgba="0.3 0.3 0.3 1" />
-            </material>
-        </visual>
-        <collision>
-            <origin xyz="0 0 0" rpy="0 0 0" />
-            <geometry>
-                <mesh filename="package://lss_arm_description/meshes/end_effector_r.STL" />
+                <mesh filename="package://lss_arm_description/meshes/visual/end_effector_r.STL" />
+            </geometry>
+            <material name="">
+                <color rgba="0.3 0.3 0.3 1" />
+            </material>
+        </visual>
+        <collision>
+            <origin xyz="0 0 0" rpy="0 0 0" />
+            <geometry>
+                <mesh filename="package://lss_arm_description/meshes/collision/end_effector_r.STL" />
             </geometry>
         </collision>
@@ -188,14 +188,14 @@
             <origin xyz="0 0 0" rpy="0 0 0" />
             <geometry>
-                <mesh filename="package://lss_arm_description/meshes/end_effector_l.STL" />
-            </geometry>
-            <material name="">
-                <color rgba="0.3 0.3 0.3 1" />
-            </material>
-        </visual>
-        <collision>
-            <origin xyz="0 0 0" rpy="0 0 0" />
-            <geometry>
-                <mesh filename="package://lss_arm_description/meshes/end_effector_l.STL" />
+                <mesh filename="package://lss_arm_description/meshes/visual/end_effector_l.STL" />
+            </geometry>
+            <material name="">
+                <color rgba="0.3 0.3 0.3 1" />
+            </material>
+        </visual>
+        <collision>
+            <origin xyz="0 0 0" rpy="0 0 0" />
+            <geometry>
+                <mesh filename="package://lss_arm_description/meshes/collision/end_effector_l.STL" />
             </geometry>
         </collision>

Commit message: Added ignition + moveit2

File: tb4_lss_arm/lss_arm_description/urdf/lss_arm/lss_arm.urdf.xacro (robot description, xacro)
@@ -4,5 +4,5 @@
      For more information, please see http://wiki.ros.org/sw_urdf_exporter -->
 <robot name="lss_4dof_arm">
-    <link name="dummy">
+    <link name="base_link">
     </link>
     <link name="link_0">
@@ -29,5 +29,5 @@
     </link>
     <joint name="dummy_joint" type="fixed">
-     <parent link="dummy"/>
+     <parent link="base_link"/>
      <child link="link_0"/>
     </joint>

File: tb4_lss_arm/lss_arm_description/urdf/tb4_lss_arm/tb4_lss_arm.urdf.xacro (robot description, xacro)
@@ -4,7 +4,23 @@
     <xacro:include filename="$(find turtlebot4_description)/urdf/lite/turtlebot4.urdf.xacro" />
     <!-- Offsets -->
-    <xacro:property name="base_rotate_z_offset"   value="${9.5*cm2m}" />
-    <xacro:property name="base_rotate_x_offset"   value="${8.5*cm2m}" />
+    <xacro:property name="base_rotate_z_offset"   value="${20*cm2m}" />
+    <xacro:property name="base_rotate_x_offset"   value="${6.3*cm2m}" />
     <!-- LSS Arm model -->
+    <link name="lss_base">
+        <visual>
+            <origin xyz="0 0 0" rpy="1.571 0 1.571" />
+            <geometry>
+                <mesh filename="package://lss_arm_description/meshes/visual/lss_base.STL" scale="0.001 0.001 0.001"/>
+            </geometry>
+            <material name="">
+                <color rgba="0.3 0.3 0.3 1" />
+            </material>
+        </visual>
+    </link>
+    <joint name="base_joint" type="fixed">
+        <parent link="base_link"/>
+        <child link="lss_base"/>
+        <origin xyz="0 0 0" rpy="0 0 0"/>
+    </joint>
     <link name="link_0">
         <inertial>
@@ -14,5 +30,5 @@
         </inertial>
         <visual>
-            <origin xyz="0 0 0" rpy="0 0 0" />
+            <origin xyz="0 0 0" rpy="0 0 1.57" />
             <geometry>
                 <mesh filename="package://lss_arm_description/meshes/visual/link_0.STL" />
@@ -23,5 +39,5 @@
         </visual>
         <collision>
-            <origin xyz="0 0 0" rpy="0 0 0" />
+            <origin xyz="0 0 0" rpy="0 0 1.57" />
             <geometry>
                 <mesh filename="package://lss_arm_description/meshes/collision/link_0.STL" />
@@ -30,5 +46,5 @@
     </link>
     <joint name="arm_base" type="fixed">
-     <parent link="base_link"/>
+     <parent link="lss_base"/>
      <child link="link_0"/>
      <origin xyz="${base_rotate_x_offset} 0 ${base_rotate_z_offset}" rpy="0 0 0"/>
