Commit message: Updated model & example

File: tb4_lss_arm/lss_ign_moveit/lss_ign_moveit2/lss_arm_description/urdf/lss_arm.urdf (robot description, URDF)
Before this commit: robot lss_arm, 9 links, 8 joints
Links:
- added link lss_arm_base_link, mass 0.05; collision mesh filename=package://lss_arm_description/meshes/collision/lss_base.STL; visual mesh filename=package://lss_arm_description/meshes/visual/lss_base.STL
- link lss_arm_end_effector_l: mass 0.0165437278185932 -> 0.0154295568992377
- link lss_arm_end_effector_r: mass 0.0166262969986533 -> 0.0152813047822834
- link lss_arm_link_0: mass 0.0745235989082936 -> 0.0717410813666018
- link lss_arm_link_1: mass 0.0658784270809996 -> 0.0628875763471834
- link lss_arm_link_2: mass 0.0616037662847113 -> 0.0592207297890142
- link lss_arm_link_3: mass 0.062951277283338 -> 0.0601490353124708
- link lss_arm_link_4: mass 0.0552917317501261 -> 0.0556319659037934
Joints:
- removed joint lss_arm_joint_base
- added joint lss_arm_base_joint: type fixed, parent world, child lss_arm_base_link, origin xyz=0 0 0 rpy=0 0 0
- added joint lss_arm_joint4: type revolute, parent lss_arm_link_3, child lss_arm_link_4, origin xyz=0.154274210199929 0.0532325846374996 0 rpy=0 0 0.332259786519651, axis 0 0 1, limit lower=-1.5707963267948966 upper=1.5707963267948966 effort=6.5687857 velocity=6.283
- joint lss_arm_joint0: axis 0 1 0 -> (none); child lss_arm_link_1 -> lss_arm_link_0; limit lower=-3.141592653589793 upper=3.141592653589793 effort=6.5687857 velocity=6.283 -> (none); origin xyz=0 0 0.0427 rpy=1.5708 0 0 -> xyz=0.063 0 0.2 rpy=0 0 0; parent lss_arm_link_0 -> lss_arm_base_link; type revolute -> fixed
- joint lss_arm_joint1: axis 0 0 1 -> 0 1 0; child lss_arm_link_2 -> lss_arm_link_1; limit lower=-1.5707963267948966 upper=1.5707963267948966 effort=6.5687857 velocity=6.283 -> lower=-3.141592653589793 upper=3.141592653589793 effort=6.5687857 velocity=6.283; origin xyz=0 0.0588000249999991 0 rpy=0 0 -1.3621104667496 -> xyz=0 0 0.042699975 rpy=1.5707963267948966 0 0; parent lss_arm_link_1 -> lss_arm_link_0
- joint lss_arm_joint2: child lss_arm_link_3 -> lss_arm_link_2; origin xyz=-0.12954806230389 0.0533975613048809 0 rpy=0 0 1.02985068022995 -> xyz=0 0.0588000249999991 0 rpy=0 0 -1.3621104667496; parent lss_arm_link_2 -> lss_arm_link_1
- joint lss_arm_joint3: child lss_arm_link_4 -> lss_arm_link_3; origin xyz=0.154274210199929 0.0532325846374996 0 rpy=0 0 0.332259786519651 -> xyz=-0.12954806230389 0.0533975613048809 0 rpy=0 0 1.02985068022995; parent lss_arm_link_3 -> lss_arm_link_2

File: tb4_lss_arm/lss_ign_moveit/lss_ign_moveit2/lss_arm_description/urdf/lss_arm.xacro (robot description, xacro)
@@ -10,15 +10,21 @@
   <!-- Properties -->
   <!--            -->
-  <xacro:property name="joint_base_name" value="joint_base"/>
+  <xacro:property name="joint_base_name" value="base_joint"/>
   <xacro:property name="joint_base_type" value="fixed"/>
+  <xacro:property name="link_base_name" value="base_link"/>
+  <xacro:property name="link_base_mu" value="0.3"/>
+  <xacro:property name="joint0_name" value="joint0"/>
+  <xacro:property name="joint0_type" value="fixed"/>
+  <xacro:property name="joint0_origin_xyz" value="0.063 0 0.2"/>
+  <xacro:property name="joint0_origin_rpy" value="0 0 0"/>
   <xacro:property name="link_0_name" value="link_0"/>
-  <xacro:property name="link_0_mu" value="247.75"/>
-  <xacro:property name="joint1_name" value="joint0"/>
+  <xacro:property name="link_0_mu" value="0.3"/>
+  <xacro:property name="joint1_name" value="joint1"/>
   <xacro:property name="joint1_type" value="revolute"/>
-  <xacro:property name="joint1_origin_xyz" value="0 0 0.0427"/>
-  <xacro:property name="joint1_origin_rpy" value="1.5708 0 0"/>
+  <xacro:property name="joint1_origin_xyz" value="0 0 0.042699975"/>
+  <xacro:property name="joint1_origin_rpy" value="${pi/2} 0 0"/>
   <xacro:property name="joint1_axis_xyz" value="0 1 0"/>
-  <xacro:property name="joint1_lower_limit" value="${-180*pi/180}"/>
-  <xacro:property name="joint1_upper_limit" value="${180*pi/180}"/>
+  <xacro:property name="joint1_lower_limit" value="${-pi}"/>
+  <xacro:property name="joint1_upper_limit" value="${pi}"/>
   <xacro:property name="joint1_velocity_limit" value="6.283"/>
   <xacro:property name="joint1_torque_limit" value="6.5687857"/>
@@ -26,12 +32,12 @@
   <xacro:property name="joint1_friction" value="3.48"/>
   <xacro:property name="link_1_name" value="link_1"/>
-  <xacro:property name="link_1_mu" value="247.75"/>
-  <xacro:property name="joint2_name" value="joint1"/>
+  <xacro:property name="link_1_mu" value="0.3"/>
+  <xacro:property name="joint2_name" value="joint2"/>
   <xacro:property name="joint2_type" value="revolute"/>
   <xacro:property name="joint2_origin_xyz" value="0 0.0588000249999991 0"/>
   <xacro:property name="joint2_origin_rpy" value="0 0 -1.3621104667496"/>
   <xacro:property name="joint2_axis_xyz" value="0 0 1"/>
-  <xacro:property name="joint2_lower_limit" value="${-90*pi/180}"/>
-  <xacro:property name="joint2_upper_limit" value="${90*pi/180}"/>
+  <xacro:property name="joint2_lower_limit" value="${-pi/2}"/>
+  <xacro:property name="joint2_upper_limit" value="${pi/2}"/>
   <xacro:property name="joint2_velocity_limit" value="6.283"/>
   <xacro:property name="joint2_torque_limit" value="6.5687857"/>
@@ -39,12 +45,12 @@
   <xacro:property name="joint2_friction" value="3.48"/>
   <xacro:property name="link_2_name" value="link_2"/>
-  <xacro:property name="link_2_mu" value="247.75"/>
-  <xacro:property name="joint3_name" value="joint2"/>
+  <xacro:property name="link_2_mu" value="0.3"/>
+  <xacro:property name="joint3_name" value="joint3"/>
   <xacro:property name="joint3_type" value="revolute"/>
   <xacro:property name="joint3_origin_xyz" value="-0.12954806230389 0.0533975613048809 0"/>
   <xacro:property name="joint3_origin_rpy" value="0 0 1.02985068022995"/>
   <xacro:property name="joint3_axis_xyz" value="0 0 1"/>
-  <xacro:property name="joint3_lower_limit" value="${-90*pi/180}"/>
-  <xacro:property name="joint3_upper_limit" value="${90*pi/180}"/>
+  <xacro:property name="joint3_lower_limit" value="${-pi/2}"/>
+  <xacro:property name="joint3_upper_limit" value="${pi/2}"/>
   <xacro:property name="joint3_velocity_limit" value="6.283"/>
   <xacro:property name="joint3_torque_limit" value="6.5687857"/>
@@ -52,12 +58,12 @@
   <xacro:property name="joint3_friction" value="3.48"/>
   <xacro:property name="link_3_name" value="link_3"/>
-  <xacro:property name="link_3_mu" value="247.75"/>
-  <xacro:property name="joint4_name" value="joint3"/>
+  <xacro:property name="link_3_mu" value="0.3"/>
+  <xacro:property name="joint4_name" value="joint4"/>
   <xacro:property name="joint4_type" value="revolute"/>
   <xacro:property name="joint4_origin_xyz" value="0.154274210199929 0.0532325846374996 0"/>
   <xacro:property name="joint4_origin_rpy" value="0 0 0.332259786519651"/>
   <xacro:property name="joint4_axis_xyz" value="0 0 1"/>
-  <xacro:property name="joint4_lower_limit" value="${-90*pi/180}"/>
-  <xacro:property name="joint4_upper_limit" value="${90*pi/180}"/>
+  <xacro:property name="joint4_lower_limit" value="${-pi/2}"/>
+  <xacro:property name="joint4_upper_limit" value="${pi/2}"/>
   <xacro:property name="joint4_velocity_limit" value="6.283"/>
   <xacro:property name="joint4_torque_limit" value="6.5687857"/>
@@ -65,5 +71,5 @@
   <xacro:property name="joint4_friction" value="3.48"/>
   <xacro:property name="link_4_name" value="link_4"/>
-  <xacro:property name="link_4_mu" value="247.75"/>
+  <xacro:property name="link_4_mu" value="0.3"/>
   <xacro:property name="gripper_name" value="gripper_link"/>
   <xacro:property name="gripper_origin_xyz" value="0 0 0"/>
@@ -92,9 +98,25 @@
     <xacro:lss_arm_joint
     parent="${base_parent}"
-    child="${prefix}${link_0_name}"
+    child="${prefix}${link_base_name}"
     joint_name="${prefix}${joint_base_name}"
     joint_type="${joint_base_type}"
     joint_origin_xyz="${origin_xyz}"
     joint_origin_rpy="${origin_rpy}"
+    gazebo_preserve_fixed_joint="${gazebo_preserve_fixed_joint}"
+    />
+    <xacro:lss_arm_link
+    link_name="${prefix}${link_base_name}"
+    mesh="${link_base_mesh}"
+    collision="${collision}"
+    mu="${link_base_mu}"
+    />
+    <!-- 0 -->
+    <xacro:lss_arm_joint
+    parent="${prefix}${link_base_name}"
+    child="${prefix}${link_0_name}"
+    joint_name="${prefix}${joint0_name}"
+    joint_type="${joint0_type}"
+    joint_origin_xyz="${joint0_origin_xyz}"
+    joint_origin_rpy="${joint0_origin_rpy}"
     gazebo_preserve_fixed_joint="${gazebo_preserve_fixed_joint}"
     />

File: tb4_lss_arm/lss_ign_moveit/lss_ign_moveit2/lss_arm_description/urdf/lss_arm_inertial.xacro (robot description, xacro)
@@ -5,4 +5,5 @@
   <!-- Properties -->
   <!--            -->
+  <xacro:property name="link_base_mesh" value="lss_base"/>
   <xacro:property name="link_0_mesh" value="link_0"/>
   <xacro:property name="link_1_mesh" value="link_1"/>
@@ -20,51 +21,58 @@
     mesh_offset_rpy:=${mesh_offset_rpy}
   ">
+    <xacro:if value="${mesh == link_base_mesh}">
+      <inertial>
+          <origin xyz="0 0 0" rpy="${mesh_offset_rpy}" />
+          <mass value="0.05" />
+          <inertia ixx="4.17127E-06" ixy="-5.07076E-17" ixz="-8.99321E-15" iyy="8.84892E-06" iyz="5.22561E-14" izz="4.67905E-06" />
+      </inertial>
+    </xacro:if>
     <xacro:if value="${mesh == link_0_mesh}">
       <inertial>
-          <origin xyz="-9.22746070072536E-09 0.00772579323332284 0.0258164486308589" rpy="${mesh_offset_rpy}" />
-          <mass value="0.0745235989082936" />
-          <inertia ixx="3.06926142332185E-05" ixy="9.19227938875618E-11" ixz="2.60960163114495E-12" iyy="2.37938175373349E-05" iyz="2.14419674075701E-07" izz="4.37402989726652E-05" />
+          <origin xyz="-2.73691915043146E-09 0.0078496161601494 0.0255901951226594" rpy="${mesh_offset_rpy}" />
+          <mass value="0.0717410813666018" />
+          <inertia ixx="3.0636904073993E-05" ixy="9.19910875697947E-11" ixz="-6.99542916495097E-14" iyy="2.37381054307842E-05" iyz="2.14417631554388E-07" izz="4.37325540149466E-05" />
       </inertial>
     </xacro:if>
     <xacro:if value="${mesh == link_1_mesh}">
       <inertial>
-          <origin xyz="1.01932002252511E-06 0.0346260395806251 0.000106547591030595" rpy="${mesh_offset_rpy}" />
-          <mass value="0.0658784270809996" />
-          <inertia ixx="2.21234278407549E-05" ixy="9.24359378260813E-11" ixz="-3.0028304734589E-12" iyy="2.30585181059312E-05" iyz="-2.19526468312218E-07" izz="1.89994043624137E-05" />
+          <origin xyz="1.5578217768027E-09 0.0348051841749016 0.00014951767591631" rpy="${mesh_offset_rpy}" />
+          <mass value="0.0628875763471834" />
+          <inertia ixx="2.20425725995968E-05" ixy="9.19935112458848E-11" ixz="1.70368679861891E-13" iyy="2.29485908974563E-05" iyz="-2.19524118186986E-07" izz="1.89578527653699E-05" />
       </inertial>
     </xacro:if>
     <xacro:if value="${mesh == link_2_mesh}">
       <inertial>
-          <origin xyz="-0.111778545935364 0.0336104387117684 0.000180852718742204" rpy="${mesh_offset_rpy}" />
-          <mass value="0.0616037662847113" />
-          <inertia ixx="1.66852308837933E-05" ixy="-1.03329219740433E-06" ixz="-4.43310654754874E-08" iyy="1.20242622304033E-05" iyz="-2.15007795219099E-07" izz="1.41673473261847E-05" />
+          <origin xyz="-0.112045323028693 0.0336416089233315 0.000234166707606796" rpy="${mesh_offset_rpy}" />
+          <mass value="0.0592207297890142" />
+          <inertia ixx="1.66333998725443E-05" ixy="-1.03352394963547E-06" ixz="-4.43274108116386E-08" iyy="1.1971383214163E-05" iyz="-2.15005479062966E-07" izz="1.41577057658295E-05" />
       </inertial>
     </xacro:if>
     <xacro:if value="${mesh == link_3_mesh}">
       <inertial>
-          <origin xyz="0.119392702406077 0.0410364992253052 0.000154048902422472" rpy="${mesh_offset_rpy}" />
-          <mass value="0.062951277283338" />
-          <inertia ixx="1.11886789972704E-05" ixy="-2.66768170363405E-06" ixz="-2.01609481649329E-07" iyy="1.79991460198167E-05" iyz="-6.9561531958934E-08" izz="1.46158276124359E-05" />
+          <origin xyz="0.119623138465818 0.0411506770766876 0.000345214465821365" rpy="${mesh_offset_rpy}" />
+          <mass value="0.0601490353124708" />
+          <inertia ixx="1.1113660383281E-05" ixy="-2.67466932607218E-06" ixz="2.01605698642722E-07" iyy="1.79419649434231E-05" iyz="-6.9564477599757E-08" izz="1.45807099366603E-05" />
       </inertial>
     </xacro:if>
     <xacro:if value="${mesh == link_4_mesh}">
       <inertial>
-          <origin xyz="0.0463345232293113 -0.000217116498809761 0.000342446314582681" rpy="${mesh_offset_rpy}" />
-          <mass value="0.0552917317501261" />
-          <inertia ixx="1.81135754161747E-05" ixy="3.0049831947197E-12" ixz="9.20482185162439E-11" iyy="1.48586070714427E-05" iyz="2.14450571018836E-07" izz="9.04738520213568E-06" />
+          <origin xyz="0.0446894562780881 -0.000131072409021604 0.000356231689785028" rpy="${mesh_offset_rpy}" />
+          <mass value="0.0556319659037934" />
+          <inertia ixx="1.81337749108788E-05" ixy="-6.99513846908487E-14" ixz="9.19941036664484E-11" iyy="1.49173144124065E-05" iyz="2.14447838213905E-07" izz="9.12796728342695E-06" />
       </inertial>
     </xacro:if>
     <xacro:if value="${mesh == end_effector_r_mesh}">
       <inertial>
-          <origin xyz="0.0308013779043008 -0.0141013526461647 0.00131237715084586" rpy="${mesh_offset_rpy}" />
-          <mass value="0.0166262969986533" />
-          <inertia ixx="6.38976786525478E-07" ixy="-1.49469409770964E-12" ixz="-4.41621752133789E-07" iyy="3.00353485001635E-06" iyz="-4.34708916625113E-12" izz="2.57289120441113E-06" />
+          <origin xyz="0.0310712366675979 -0.0140452526813673 0.00133953163684892" rpy="${mesh_offset_rpy}" />
+          <mass value="0.0152813047822834" />
+          <inertia ixx="6.12119941271843E-07" ixy="-1.61044889315886E-12" ixz="-4.41621763353496E-07" iyy="2.99804070646807E-06" iyz="-3.8879675590965E-12" izz="2.54603357212087E-06" />
       </inertial>
     </xacro:if>
     <xacro:if value="${mesh == end_effector_l_mesh}">
       <inertial>
-          <origin xyz="0.0309551132879063 -0.0140672528822861 -0.0013189270605785" rpy="${mesh_offset_rpy}" />
-          <mass value="0.0165437278185932" />
-          <inertia ixx="6.37840843695913E-07" ixy="-1.67462842205218E-12" ixz="4.41621808330111E-07" iyy="3.00246171921638E-06" iyz="3.99757576475728E-12" izz="2.57175512278327E-06" />
+          <origin xyz="0.0307726942893274 -0.0140975049159748 -0.0013266609885073" rpy="${mesh_offset_rpy}" />
+          <mass value="0.0154295568992377" />
+          <inertia ixx="6.13242885883712E-07" ixy="-1.69555790218149E-12" ixz="4.41621764601781E-07" iyy="2.99899721506146E-06" iyz="4.09343888509186E-12" izz="2.54715653674288E-06" />
       </inertial>
     </xacro:if>

File: tb4_lss_arm/lss_ign_moveit/lss_ign_moveit2/lss_arm_description/urdf/lss_gripper.xacro (robot description, xacro)
@@ -10,8 +10,4 @@
   <!-- Properties -->
   <!--            -->
-  <!-- <xacro:property name="joint_gripper_name" value="joint_gripper"/>
-  <xacro:property name="joint_gripper_type" value="fixed"/>
-  <xacro:property name="hand_name" value="hand"/>
-  <xacro:property name="hand_mu" value="0.85"/> -->
   <xacro:property name="joint_finger1_name" value="gripper_r"/>
   <xacro:property name="joint_finger1_type" value="revolute"/>
@@ -20,5 +16,5 @@
   <xacro:property name="joint_finger1_axis_xyz" value="0 1 0"/>
   <xacro:property name="joint_finger1_lower_limit" value="0"/>
-  <xacro:property name="joint_finger1_upper_limit" value="${90*pi/180}"/>
+  <xacro:property name="joint_finger1_upper_limit" value="${pi/2}"/>
   <xacro:property name="joint_finger1_velocity_limit" value="6.283"/>
   <xacro:property name="joint_finger1_torque_limit" value="6.5687857"/>
@@ -26,5 +22,5 @@
   <xacro:property name="joint_finger1_friction" value="0.4"/>
   <xacro:property name="link_finger1_name" value="end_effector_r"/>
-  <xacro:property name="link_finger1_mu" value="247.75"/>
+  <xacro:property name="link_finger1_mu" value="0.3"/>
   <xacro:property name="link_finger1_mesh_offset" value="0 0 0"/>
   <xacro:property name="joint_finger2_name" value="gripper_l"/>
@@ -33,5 +29,5 @@
   <xacro:property name="joint_finger2_origin_rpy" value="0 0 0"/>
   <xacro:property name="joint_finger2_axis_xyz" value="0 1 0"/>
-  <xacro:property name="joint_finger2_lower_limit" value="${-90*pi/180}"/>
+  <xacro:property name="joint_finger2_lower_limit" value="${-pi/2}"/>
   <xacro:property name="joint_finger2_upper_limit" value="0"/>
   <xacro:property name="joint_finger2_velocity_limit" value="6.283"/>
@@ -40,5 +36,5 @@
   <xacro:property name="joint_finger2_friction" value="0.4"/>
   <xacro:property name="link_finger2_name" value="end_effector_l"/>
-  <xacro:property name="link_finger2_mu" value="247.75"/>
+  <xacro:property name="link_finger2_mu" value="0.3"/>
   <xacro:property name="link_finger2_mesh_offset" value="0 0 0"/>
   <xacro:property name="ee_name" value="hand_tcp"/>

File: tb4_lss_arm/lss_ign_moveit/lss_ign_moveit2/lss_arm_moveit/srdf/lss_arm.xacro (robot description, xacro)
@@ -11,8 +11,8 @@
     </group>
     <group_state group="lss_arm" name="home" >
-        <joint name="${prefix}joint0" value="0.0"/>
         <joint name="${prefix}joint1" value="0.0"/>
-        <joint name="${prefix}joint2" value="0.0"/>
-        <joint name="${prefix}joint3" value="0.0"/>
+        <joint name="${prefix}joint2" value="0.8"/>
+        <joint name="${prefix}joint3" value="-0.4"/>
+        <joint name="${prefix}joint4" value="-0.4"/>
     </group_state>
     <disable_collisions link1="${prefix}link_0" link2="${prefix}link_1" reason="Adjacent"/>
