Commit message: Added version w/ TB4+LSS Arm

File: tb4_lss_arm/lss_ign_moveit/lss_ign_moveit2/lss_arm_description/urdf/lss_arm.urdf (robot description, URDF)
Before this commit: robot lss_arm, 10 links, 9 joints
Links:
- removed link lss_arm_base_link
Joints:
- removed joint lss_arm_base_joint
- joint lss_arm_joint0: origin xyz=0.063 0 0.2 rpy=0 0 0 -> xyz=0 0 0 rpy=0 0 0; parent lss_arm_base_link -> world

File: tb4_lss_arm/lss_ign_moveit/lss_ign_moveit2/lss_arm_description/urdf/lss_arm.xacro (robot description, xacro)
@@ -10,11 +10,18 @@
   <!-- Properties -->
   <!--            -->
-  <xacro:property name="joint_base_name" value="base_joint"/>
-  <xacro:property name="joint_base_type" value="fixed"/>
-  <xacro:property name="link_base_name" value="base_link"/>
-  <xacro:property name="link_base_mu" value="0.3"/>
+  <xacro:unless value="$(arg tb4)">
+    <xacro:property name="link_base_name" value="world"/>
+  </xacro:unless>
+  <xacro:if value="$(arg tb4)">
+    <xacro:property name="link_base_name" value="lss_arm_base_link"/>
+  </xacro:if>
   <xacro:property name="joint0_name" value="joint0"/>
   <xacro:property name="joint0_type" value="fixed"/>
-  <xacro:property name="joint0_origin_xyz" value="0.063 0 0.2"/>
+  <xacro:unless value="$(arg tb4)">
+    <xacro:property name="joint0_origin_xyz" value="0 0 0"/>
+  </xacro:unless>
+  <xacro:if value="$(arg tb4)">
+    <xacro:property name="joint0_origin_xyz" value="0.063 0 0.2"/>
+  </xacro:if>
   <xacro:property name="joint0_origin_rpy" value="0 0 0"/>
   <xacro:property name="link_0_name" value="link_0"/>
@@ -75,43 +82,27 @@
   <xacro:property name="gripper_origin_xyz" value="0 0 0"/>
   <xacro:property name="gripper_origin_rpy" value="0 0 0"/>
-  <!--       -->
-  <!-- Macro -->
-  <!--       -->
-  <xacro:property name="default_origin_xyz" value="0 0 0"/>
-  <xacro:property name="default_origin_rpy" value="0 0 0"/>
-  <xacro:macro name="lss_arm" params="
-    base_parent
-    prefix
-    origin_xyz:=${default_origin_xyz}
-    origin_rpy:=${default_origin_rpy}
-    collision:=true
-    safety_limits:=false
-    safety_position_margin:=${pi/180}
-    safety_k_position:=100.0
-    safety_k_velocity:=40.0
-    ros2_control:=true
-    ros2_control_plugin:=fake
-    ros2_control_command_interface:=effort
-    gazebo_preserve_fixed_joint:=false
-  ">
-    <!-- Base -->
-    <xacro:lss_arm_joint
-    parent="${base_parent}"
-    child="${prefix}${link_base_name}"
-    joint_name="${prefix}${joint_base_name}"
-    joint_type="${joint_base_type}"
-    joint_origin_xyz="${origin_xyz}"
-    joint_origin_rpy="${origin_rpy}"
-    gazebo_preserve_fixed_joint="${gazebo_preserve_fixed_joint}"
-    />
-    <xacro:lss_arm_link
-    link_name="${prefix}${link_base_name}"
-    mesh="${link_base_mesh}"
-    collision="${collision}"
-    mu="${link_base_mu}"
-    />
+    <!--       -->
+    <!-- Macro -->
+    <!--       -->
+    <xacro:property name="default_origin_xyz" value="0 0 0"/>
+    <xacro:property name="default_origin_rpy" value="0 0 0"/>
+    <xacro:macro name="lss_arm" params="
+      base_parent
+      prefix
+      origin_xyz:=${default_origin_xyz}
+      origin_rpy:=${default_origin_rpy}
+      collision:=true
+      safety_limits:=false
+      safety_position_margin:=${pi/180}
+      safety_k_position:=100.0
+      safety_k_velocity:=40.0
+      ros2_control:=true
+      ros2_control_plugin:=fake
+      ros2_control_command_interface:=effort
+      gazebo_preserve_fixed_joint:=false
+    ">
     <!-- 0 -->
     <xacro:lss_arm_joint
-    parent="${prefix}${link_base_name}"
+    parent="${link_base_name}"
     child="${prefix}${link_0_name}"
     joint_name="${prefix}${joint0_name}"

File: tb4_lss_arm/lss_ign_moveit/lss_ign_moveit2/lss_arm_description/urdf/tb4_lss_arm.urdf.xacro (robot description, xacro)
@@ -5,4 +5,5 @@
   <!-- Imported elements -->
   <!--                   -->
+  <xacro:include filename="$(find lss_arm_description)/urdf/tb4_base.xacro"/>
   <xacro:include filename="$(find lss_arm_description)/urdf/lss_arm.xacro"/>
   <xacro:include filename="$(find lss_arm_description)/urdf/lss_gripper.xacro"/>
@@ -12,12 +13,14 @@
   <!-- Parameters -->
   <!--            -->
-  <!-- Flag to enable tb4 bracket -->
+  <!-- Flag to enable tb4 platform -->
   <xacro:arg name="tb4" default="true" />
   <!-- Name of the robot (mandatory) -->
-  <xacro:arg name="name" default="lss_arm"/>
+  <xacro:arg name="name" default="tb4_lss_arm"/>
   <!-- Prefix for all entities -->
   <xacro:arg name="prefix" default="lss_arm_"/>
   <!-- Flag to enable default gripper -->
   <xacro:arg name="gripper" default="true" />
+  <!-- Flag to enable collision geometry for TB4 platform -->
+  <xacro:arg name="collision_tb4" default="true"/>
   <!-- Flag to enable collision geometry for manipulator's arm -->
   <xacro:arg name="collision_arm" default="true"/>
@@ -63,7 +66,20 @@
     gazebo_preserve_fixed_joint="$(arg gazebo_preserve_fixed_joint)"
   />
+  <!-- TB4 Platform -->
+  <xacro:tb4_base
+    base_parent="${world_name}"
+    prefix="${prefix_arm}"
+    origin_xyz="${origin_xyz}"
+    origin_rpy="${origin_rpy}"
+    collision="$(arg collision_tb4)"
+    safety_limits="$(arg safety_limits)"
+    ros2_control="$(arg ros2_control)"
+    ros2_control_plugin="$(arg ros2_control_plugin)"
+    ros2_control_command_interface="$(arg ros2_control_command_interface)"
+    gazebo_preserve_fixed_joint="$(arg gazebo_preserve_fixed_joint)"
+  />
   <!-- Arm -->
   <xacro:lss_arm
-    base_parent="${world_name}"
+    base_parent="base_link"
     prefix="${prefix_arm}"
     origin_xyz="${origin_xyz}"
