Commit message: Added 5DoF model

File: lss_arm_description/urdf/lss_arm.urdf.xacro (robot description, xacro)
@@ -1,27 +1,24 @@
 <?xml version="1.0"?>
-<!-- URDF for LSS 4DoF Arm -->
+<!-- URDF for LSS 4DoF/5DoF Arms -->
 <robot xmlns:xacro="http://wiki.ros.org/xacro" name="$(arg name)">
   <!--                   -->
   <!-- Imported elements -->
   <!--                   -->
-  <xacro:include filename="$(find lss_arm_description)/urdf/lss_arm.xacro"/>
-  <xacro:include filename="$(find lss_arm_description)/urdf/lss_gripper.xacro"/>
   <xacro:include filename="$(find lss_arm_description)/urdf/lss_arm_utils.xacro"/>
   <xacro:include filename="$(find lss_arm_description)/urdf/lss_arm.gazebo"/>
+  <xacro:include filename="$(find lss_arm_description)/urdf/lss_arm.xacro"/>
   <!--            -->
   <!-- Parameters -->
   <!--            -->
-  <!-- Flag to enable tb4 platform -->
-  <xacro:arg name="tb4" default="false" />
+  <!-- Flag to enable adapter_bracket platform -->
+  <xacro:arg name="adapter_bracket" default="false" />
+  <!-- Parameter to select gripper model-->
+  <xacro:arg name="dof" default="4"/>
   <!-- Name of the robot (mandatory) -->
   <xacro:arg name="name" default="lss_arm"/>
   <!-- Prefix for all entities -->
   <xacro:arg name="prefix" default="lss_arm_"/>
-  <!-- Flag to enable default gripper -->
-  <xacro:arg name="gripper" default="true" />
   <!-- Flag to enable collision geometry for manipulator's arm -->
-  <xacro:arg name="collision_arm" default="true"/>
-  <!-- Flag to enable collision geometry for manipulator's gripper (hand and fingers) -->
-  <xacro:arg name="collision_gripper" default="true"/>
+  <xacro:arg name="collision" default="true"/>
   <!-- Flag to enable safety limits controllers on manipulator joints -->
   <xacro:arg name="safety_limits" default="false"/>
@@ -36,8 +33,6 @@
   <!-- The ros2_control plugin that should be loaded for the manipulator ('fake', 'ign', 'real' or custom) -->
   <xacro:arg name="ros2_control_plugin" default="ign"/>
-  <!-- The output control command interface provided by ros2_control ('position', 'velocity', 'effort' or certain combinations 'position,velocity') -->
-  <xacro:arg name="ros2_control_command_interface" default="position"/>
   <!-- The filepath to parameters of ROS 2 controllers -->
-  <xacro:arg name="ros2_controller_parameters" default="$(find lss_arm_moveit)/config/controllers_$(arg ros2_control_command_interface).yaml"/>
+  <xacro:arg name="ros2_controller_parameters" default="$(find lss_arm_moveit)/config/controllers_$(arg dof)dof.yaml"/>
   <!-- Flag to preserve fixed joints and prevent lumping when generating SDF for Gazebo -->
   <xacro:arg name="gazebo_preserve_fixed_joint" default="false"/>
@@ -47,5 +42,4 @@
   <!-- Prefixes -->
   <xacro:property name="prefix_arm" value="$(arg prefix)"/>
-  <xacro:property name="prefix_gripper" value="$(arg prefix)"/>
   <!-- Origin of robot in the world -->
   <xacro:property name="world_name" value="world"/>
@@ -63,8 +57,8 @@
     gazebo_preserve_fixed_joint="$(arg gazebo_preserve_fixed_joint)"
   />
-  <xacro:unless value="$(arg tb4)">
+  <xacro:unless value="$(arg adapter_bracket)">
     <xacro:property name="joint_0_origin_xyz" value="0 0 0"/>
   </xacro:unless>
-  <xacro:if value="$(arg tb4)">
+  <xacro:if value="$(arg adapter_bracket)">
     <xacro:property name="joint_0_origin_xyz" value="0.063 0 0.2"/>
   </xacro:if>
@@ -75,5 +69,5 @@
     origin_xyz="${origin_xyz}"
     origin_rpy="${origin_rpy}"
-    collision="$(arg collision_arm)"
+    collision="$(arg collision)"
     safety_limits="$(arg safety_limits)"
     safety_position_margin="$(arg safety_position_margin)"
@@ -82,18 +76,38 @@
     ros2_control="$(arg ros2_control)"
     ros2_control_plugin="$(arg ros2_control_plugin)"
-    ros2_control_command_interface="$(arg ros2_control_command_interface)"
     gazebo_preserve_fixed_joint="$(arg gazebo_preserve_fixed_joint)"
   />
   <!-- Gripper -->
-  <xacro:if value="$(arg gripper)">
-    <xacro:lss_gripper
-      lss_gripper="${prefix_arm}${gripper_name}"
-      prefix="${prefix_gripper}"
+  <xacro:if value="${'$(arg dof)' == '4'}">
+  <xacro:include filename="$(find lss_arm_description)/urdf/lss_gripper_4dof.xacro"/>
+    <xacro:gripper_4dof
+      lss_gripper="${prefix_arm}gripper_4dof"
+      prefix="${prefix_arm}"
       origin_xyz="${gripper_offset_xyz}"
       origin_rpy="${gripper_offset_rpy}"
-      collision="$(arg collision_gripper)"
+      collision="$(arg collision)"
+      safety_limits="$(arg safety_limits)"
+      safety_position_margin="$(arg safety_position_margin)"
+      safety_k_position="$(arg safety_k_position)"
+      safety_k_velocity="$(arg safety_k_velocity)"
       ros2_control="$(arg ros2_control)"
       ros2_control_plugin="$(arg ros2_control_plugin)"
-      ros2_control_command_interface="$(arg ros2_control_command_interface)"
+      gazebo_preserve_fixed_joint="$(arg gazebo_preserve_fixed_joint)"
+    />
+  </xacro:if>
+  <xacro:if value="${'$(arg dof)' == '5'}">
+  <xacro:include filename="$(find lss_arm_description)/urdf/lss_gripper_5dof.xacro"/>
+    <xacro:gripper_5dof
+      lss_gripper="${prefix_arm}gripper_5dof"
+      prefix="${prefix_arm}"
+      origin_xyz="${gripper_offset_xyz}"
+      origin_rpy="${gripper_offset_rpy}"
+      collision="$(arg collision)"
+      safety_limits="$(arg safety_limits)"
+      safety_position_margin="$(arg safety_position_margin)"
+      safety_k_position="$(arg safety_k_position)"
+      safety_k_velocity="$(arg safety_k_velocity)"
+      ros2_control="$(arg ros2_control)"
+      ros2_control_plugin="$(arg ros2_control_plugin)"
       gazebo_preserve_fixed_joint="$(arg gazebo_preserve_fixed_joint)"
     />

File: lss_arm_description/urdf/lss_arm.xacro (robot description, xacro)
@@ -1,4 +1,4 @@
 <?xml version="1.0"?>
-<!-- Xacro for LSS 4DoF Arm -->
+<!-- Xacro for LSS Arms -->
 <robot xmlns:xacro="http://www.ros.org/wiki/xacro">
   <!--                   -->
@@ -54,20 +54,4 @@
   <xacro:property name="link_3_name" value="link_3"/>
   <xacro:property name="link_3_mu" value="0.3"/>
-  <xacro:property name="joint_4_name" value="joint_4"/>
-  <xacro:property name="joint_4_type" value="revolute"/>
-  <xacro:property name="joint_4_origin_xyz" value="0.154274210199929 0.0532325846374996 0"/>
-  <xacro:property name="joint_4_origin_rpy" value="0 0 0.332259786519651"/>
-  <xacro:property name="joint_4_axis_xyz" value="0 0 1"/>
-  <xacro:property name="joint_4_lower_limit" value="${-110*pi/180}"/>
-  <xacro:property name="joint_4_upper_limit" value="${110*pi/180}"/>
-  <xacro:property name="joint_4_velocity_limit" value="6.283"/>
-  <xacro:property name="joint_4_torque_limit" value="6.8439285"/>
-  <xacro:property name="joint_4_damping" value="0.01"/>
-  <xacro:property name="joint_4_friction" value="3.48"/>
-  <xacro:property name="link_4_name" value="link_4"/>
-  <xacro:property name="link_4_mu" value="0.3"/>
-  <xacro:property name="gripper_name" value="joint_gripper"/>
-  <xacro:property name="gripper_origin_xyz" value="0 0 0"/>
-  <xacro:property name="gripper_origin_rpy" value="0 0 0"/>
     <!--       -->
     <!-- Macro -->
@@ -87,5 +71,4 @@
       ros2_control:=true
       ros2_control_plugin:=fake
-      ros2_control_command_interface:=position
       gazebo_preserve_fixed_joint:=false
     ">
@@ -187,34 +170,7 @@
     mu="${link_3_mu}"
     />
-    <!-- 4 -->
-    <xacro:lss_arm_joint_
-    parent="${prefix}${link_3_name}"
-    child="${prefix}${link_4_name}"
-    joint_name="${prefix}${joint_4_name}"
-    joint_type="${joint_4_type}"
-    joint_origin_xyz="${joint_4_origin_xyz}"
-    joint_origin_rpy="${joint_4_origin_rpy}"
-    joint_axis_xyz="${joint_4_axis_xyz}"
-    joint_lower_limit="${joint_4_lower_limit}"
-    joint_upper_limit="${joint_4_upper_limit}"
-    joint_velocity_limit="${joint_4_velocity_limit}"
-    joint_torque_limit="${joint_4_torque_limit}"
-    joint_damping="${joint_4_damping}"
-    joint_friction="${joint_4_friction}"
-    safety_limits="${safety_limits}"
-    safety_position_margin="${safety_position_margin}"
-    safety_k_position="${safety_k_position}"
-    safety_k_velocity="${safety_k_velocity}"
-    gazebo_preserve_fixed_joint="${gazebo_preserve_fixed_joint}"
-    />
-    <xacro:lss_arm_link
-    link_name="${prefix}${link_4_name}"
-    mesh="${link_4_mesh}"
-    collision="${collision}"
-    mu="${link_4_mu}"
-    />
-    <!-- ROS 2 control -->
+     <!-- ROS 2 control -->
     <xacro:if value="${ros2_control}">
-      <xacro:ros2_control_lss_arm prefix="${prefix}" plugin="${ros2_control_plugin}" command_interface="${ros2_control_command_interface}"/>
+        <xacro:ros2_control_lss_arm prefix="${prefix}" plugin="${ros2_control_plugin}" command_interface="position"/>
     </xacro:if>
   </xacro:macro>

File: lss_arm_description/urdf/lss_arm_inertial.xacro (robot description, xacro)
@@ -10,7 +10,9 @@
   <xacro:property name="link_2_mesh" value="link_2"/>
   <xacro:property name="link_3_mesh" value="link_3"/>
-  <xacro:property name="link_4_mesh" value="link_4"/>
+  <xacro:property name="link_4_mesh_4dof" value="link_4_4dof"/>
+  <xacro:property name="link_4_mesh_5dof" value="link_4_5dof"/>
+  <xacro:property name="link_5_mesh_5dof" value="link_5_5dof"/>
+  <xacro:property name="finger_l_mesh" value="finger_l"/>
   <xacro:property name="finger_r_mesh" value="finger_r"/>
-  <xacro:property name="finger_l_mesh" value="finger_l"/>
   <!--       -->
   <!-- Macro -->
@@ -56,5 +58,5 @@
       </inertial>
     </xacro:if>
-    <xacro:if value="${mesh == link_4_mesh}">
+    <xacro:if value="${mesh == link_4_mesh_4dof}">
       <inertial>
           <origin xyz="0.0446894562780881 -0.000131072409021604 0.000356231689785028" rpy="${mesh_offset_rpy}" />
@@ -63,5 +65,19 @@
       </inertial>
     </xacro:if>
-    <xacro:if value="${mesh == finger_r_mesh}">
+    <xacro:if value="${mesh == link_4_mesh_5dof}">
+      <inertial>
+          <origin xyz="0.041227 -1.5305E-06 -0.010489" rpy="${mesh_offset_rpy}" />
+          <mass value="0.051733" />
+          <inertia ixx="1.3345E-05" ixy="2.5814E-10" ixz="-1.8101E-07" iyy="1.6468E-05" iyz="-7.6602E-10" izz="8.1683E-06" />
+      </inertial>
+    </xacro:if>
+    <xacro:if value="${mesh == link_5_mesh_5dof}">
+      <inertial>
+          <origin xyz="0.033089 -0.0086089 4.6839E-05" rpy="${mesh_offset_rpy}" />
+          <mass value="0.050102" />
+          <inertia ixx="1.6176E-05" ixy="-9.3694E-14" ixz="9.1972E-11" iyy="1.2688E-05" iyz="2.1445E-07" izz="8.3014E-06" />
+      </inertial>
+    </xacro:if>
+    <xacro:if value="${mesh == finger_l_mesh}">
       <inertial>
           <origin xyz="0.0310712366675979 -0.0140452526813673 0.00133953163684892" rpy="${mesh_offset_rpy}" />
@@ -70,5 +86,5 @@
       </inertial>
     </xacro:if>
-    <xacro:if value="${mesh == finger_l_mesh}">
+    <xacro:if value="${mesh == finger_r_mesh}">
       <inertial>
           <origin xyz="0.0307726942893274 -0.0140975049159748 -0.0013266609885073" rpy="${mesh_offset_rpy}" />

File: lss_arm_description/urdf/lss_arm_utils.xacro (robot description, xacro)
@@ -11,5 +11,5 @@
   <xacro:macro name="DarkGreyMaterial">
     <material name="DarkGrey">
-      <color rgba="0.3 0.3 0.3 1.0"/>
+      <color rgba="0.75294 0.75294 0.75294 1.0"/>
       <diffuse>${3/255} ${3/255} ${3/255} 1</diffuse>
       <specular>0 0 0 1</specular>
@@ -191,5 +191,5 @@
   <!-- Macro -->
   <!--       -->
-  <xacro:macro name="tb4_base_virtual_link" params="
+  <xacro:macro name="adapter_bracket_base_virtual_link" params="
     parent
     link_name
@@ -198,5 +198,5 @@
     gazebo_preserve_fixed_joint:=false
   ">
-    <xacro:tb4_dummy_link
+    <xacro:adapter_bracket_dummy_link
       link_name="${parent}"
       gazebo_preserve_fixed_joint="${gazebo_preserve_fixed_joint}"
@@ -208,5 +208,5 @@
     </joint>
   </xacro:macro>
-  <xacro:macro name="tb4_dummy_link" params="
+  <xacro:macro name="adapter_bracket_dummy_link" params="
     link_name
     gazebo_preserve_fixed_joint:=false

File: lss_arm_moveit/srdf/lss_arm.srdf.xacro (robot description, xacro)
@@ -9,5 +9,5 @@
   <!--                   -->
   <xacro:include filename="$(find lss_arm_moveit)/srdf/lss_arm.xacro" />
-  <xacro:include filename="$(find lss_arm_moveit)/srdf/lss_arm_gripper.xacro" />
+  <xacro:include filename="$(find lss_arm_moveit)/srdf/lss_gripper.xacro" />
   <!--            -->
   <!-- Parameters -->
@@ -17,44 +17,39 @@
   <!-- Prefix for all entities -->
   <xacro:arg name="prefix" default="$(arg name)_"/>
+  <!-- Parameter to select gripper model-->
+  <xacro:arg name="dof" default="4"/>
   <!--            -->
   <!-- Properties -->
   <!--            -->
-  <!-- Prefixes -->
-  <xacro:property name="prefix_arm" value="$(arg prefix)"/>
-  <xacro:property name="prefix_gripper" value="$(arg prefix)"/>
+  <!--  Prefixes  -->
+  <xacro:property name="prefix" value="$(arg prefix)"/>
   <!--       -->
   <!-- Robot -->
   <!--       -->
-  <xacro:lss_arm
-    prefix="${prefix_arm}"
-  />
-  <xacro:lss_arm_gripper
-    prefix="${prefix_gripper}"
-  />
-  <group name="full_arm">
-    <group name="lss_arm"/>
-    <group name="gripper"/>
-  </group>
-  <group_state group="full_arm" name="home_close">
-    <joint name="lss_arm_joint_1" value="0.0"/>
-    <joint name="lss_arm_joint_2" value="2"/>
-    <joint name="lss_arm_joint_3" value="-0.9"/>
-    <joint name="lss_arm_joint_4" value="-1.7"/>
-    <joint name="lss_arm_joint_5" value="0.0"/>
-    <joint name="lss_arm_joint_6" value="0.0"/>
-  </group_state>
-  <group_state group="full_arm" name="home_open">
-    <joint name="lss_arm_joint_1" value="0.0"/>
-    <joint name="lss_arm_joint_2" value="2"/>
-    <joint name="lss_arm_joint_3" value="-0.9"/>
-    <joint name="lss_arm_joint_4" value="-1.7"/>
-    <joint name="lss_arm_joint_5" value="0.785"/>
-    <joint name="lss_arm_joint_6" value="-0.785"/>
-  </group_state>
-  <end_effector group="gripper" name="gripper" parent_group="lss_arm" parent_link="lss_arm_ee"/>
-  <disable_collisions link1="lss_arm_finger_l" link2="lss_arm_finger_r" reason="Default"/>
-  <disable_collisions link1="lss_arm_finger_l" link2="lss_arm_link_3" reason="Never"/>
-  <disable_collisions link1="lss_arm_finger_l" link2="lss_arm_link_4" reason="Adjacent"/>
-  <disable_collisions link1="lss_arm_finger_r" link2="lss_arm_link_3" reason="Never"/>
-  <disable_collisions link1="lss_arm_finger_r" link2="lss_arm_link_4" reason="Adjacent"/>
+  <xacro:if value="${'$(arg dof)' == '4'}">
+    <xacro:lss_arm_4dof
+      prefix="${prefix}"
+    />
+    <xacro:gripper_4dof
+      prefix="${prefix}"
+    />
+    <disable_collisions link1="${prefix}finger_r" link2="${prefix}link_3" reason="Never"/>
+    <disable_collisions link1="${prefix}finger_r" link2="${prefix}link_4" reason="Adjacent"/>
+    <disable_collisions link1="${prefix}finger_l" link2="${prefix}link_3" reason="Never"/>
+    <disable_collisions link1="${prefix}finger_l" link2="${prefix}link_4" reason="Adjacent"/>
+  </xacro:if>
+  <xacro:if value="${'$(arg dof)' == '5'}">
+    <xacro:lss_arm_5dof
+      prefix="${prefix}"
+    />
+    <xacro:gripper_5dof
+      prefix="${prefix}"
+    />
+    <disable_collisions link1="${prefix}finger_r" link2="${prefix}link_4" reason="Never"/>
+    <disable_collisions link1="${prefix}finger_r" link2="${prefix}link_5" reason="Adjacent"/>
+    <disable_collisions link1="${prefix}finger_l" link2="${prefix}link_4" reason="Never"/>
+    <disable_collisions link1="${prefix}finger_l" link2="${prefix}link_5" reason="Adjacent"/>
+  </xacro:if>
+  <end_effector group="gripper" name="gripper" parent_group="lss_arm" parent_link="${prefix}ee"/>
+  <disable_collisions link1="${prefix}finger_r" link2="${prefix}finger_l" reason="Default"/>
 </robot>

File: lss_arm_moveit/srdf/lss_arm.xacro (robot description, xacro)
@@ -4,21 +4,41 @@
   <!-- Macro -->
   <!--       -->
-  <xacro:macro name="lss_arm" params="
+  <xacro:macro name="lss_arm_4dof" params="
     prefix:=lss_arm_
   ">
     <group name="lss_arm">
-        <chain base_link="lss_arm_link_0" tip_link="lss_arm_ee"/>
+        <chain base_link="${prefix}link_0" tip_link="${prefix}ee"/>
     </group>
     <group_state group="lss_arm" name="home" >
-        <joint name="lss_arm_joint_1" value="0.0"/>
-        <joint name="lss_arm_joint_2" value="1.7"/>
-        <joint name="lss_arm_joint_3" value="-0.7"/>
-        <joint name="lss_arm_joint_4" value="-1.7"/>
+        <joint name="${prefix}joint_1" value="0.0"/>
+        <joint name="${prefix}joint_2" value="1.7"/>
+        <joint name="${prefix}joint_3" value="-0.7"/>
+        <joint name="${prefix}joint_4" value="-1.7"/>
     </group_state>
-    <disable_collisions link1="lss_arm_link_0" link2="lss_arm_link_1" reason="Adjacent"/>
-    <disable_collisions link1="lss_arm_link_0" link2="lss_arm_link_2" reason="Never"/>
-    <disable_collisions link1="lss_arm_link_1" link2="lss_arm_link_2" reason="Adjacent"/>
-    <disable_collisions link1="lss_arm_link_2" link2="lss_arm_link_3" reason="Adjacent"/>
-    <disable_collisions link1="lss_arm_link_3" link2="lss_arm_link_4" reason="Adjacent"/>
+    <disable_collisions link1="${prefix}link_0" link2="${prefix}link_1" reason="Adjacent"/>
+    <disable_collisions link1="${prefix}link_0" link2="${prefix}link_2" reason="Never"/>
+    <disable_collisions link1="${prefix}link_1" link2="${prefix}link_2" reason="Adjacent"/>
+    <disable_collisions link1="${prefix}link_2" link2="${prefix}link_3" reason="Adjacent"/>
+    <disable_collisions link1="${prefix}link_3" link2="${prefix}link_4" reason="Adjacent"/>
+  </xacro:macro>
+  <xacro:macro name="lss_arm_5dof" params="
+    prefix:=lss_arm_
+  ">
+    <group name="lss_arm">
+        <chain base_link="${prefix}link_0" tip_link="${prefix}ee"/>
+    </group>
+    <group_state group="lss_arm" name="home" >
+        <joint name="${prefix}joint_1" value="0.0"/>
+        <joint name="${prefix}joint_2" value="1.7"/>
+        <joint name="${prefix}joint_3" value="-0.7"/>
+        <joint name="${prefix}joint_4" value="-1.7"/>
+        <joint name="${prefix}joint_6" value="0.0"/>
+    </group_state>
+    <disable_collisions link1="${prefix}link_0" link2="${prefix}link_1" reason="Adjacent"/>
+    <disable_collisions link1="${prefix}link_0" link2="${prefix}link_2" reason="Never"/>
+    <disable_collisions link1="${prefix}link_1" link2="${prefix}link_2" reason="Adjacent"/>
+    <disable_collisions link1="${prefix}link_2" link2="${prefix}link_3" reason="Adjacent"/>
+    <disable_collisions link1="${prefix}link_3" link2="${prefix}link_4" reason="Adjacent"/>
+    <disable_collisions link1="${prefix}link_4" link2="${prefix}link_5" reason="Adjacent"/>
   </xacro:macro>
 </robot>
