Commit message: Adjusted limits

File: lss_arm_description/urdf/lss_arm.xacro (robot description, xacro)
@@ -23,5 +23,5 @@
   <xacro:property name="joint_1_upper_limit" value="${pi}"/>
   <xacro:property name="joint_1_velocity_limit" value="6.283"/>
-  <xacro:property name="joint_1_torque_limit" value="6.8439285"/>
+  <xacro:property name="joint_1_torque_limit" value="6.5"/>
   <xacro:property name="joint_1_damping" value="0.01"/>
   <xacro:property name="joint_1_friction" value="3.48"/>
@@ -36,5 +36,5 @@
   <xacro:property name="joint_2_upper_limit" value="${125*pi/180}"/>
   <xacro:property name="joint_2_velocity_limit" value="6.283"/>
-  <xacro:property name="joint_2_torque_limit" value="6.8439285"/>
+  <xacro:property name="joint_2_torque_limit" value="6.5"/>
   <xacro:property name="joint_2_damping" value="0.01"/>
   <xacro:property name="joint_2_friction" value="3.48"/>
@@ -49,5 +49,5 @@
   <xacro:property name="joint_3_upper_limit" value="${90*pi/180}"/>
   <xacro:property name="joint_3_velocity_limit" value="6.283"/>
-  <xacro:property name="joint_3_torque_limit" value="6.8439285"/>
+  <xacro:property name="joint_3_torque_limit" value="6.5"/>
   <xacro:property name="joint_3_damping" value="0.01"/>
   <xacro:property name="joint_3_friction" value="3.48"/>

File: lss_arm_description/urdf/lss_gripper_4dof.xacro (robot description, xacro)
@@ -17,5 +17,5 @@
   <xacro:property name="joint_4_upper_limit" value="${120*pi/180}"/>
   <xacro:property name="joint_4_velocity_limit" value="6.283"/>
-  <xacro:property name="joint_4_torque_limit" value="6.8439285"/>
+  <xacro:property name="joint_4_torque_limit" value="6.5"/>
   <xacro:property name="joint_4_damping" value="0.01"/>
   <xacro:property name="joint_4_friction" value="3.48"/>

File: lss_arm_description/urdf/lss_gripper_5dof.xacro (robot description, xacro)
@@ -17,5 +17,5 @@
   <xacro:property name="joint_4_upper_limit" value="${140*pi/180}"/>
   <xacro:property name="joint_4_velocity_limit" value="6.283"/>
-  <xacro:property name="joint_4_torque_limit" value="6.8439285"/>
+  <xacro:property name="joint_4_torque_limit" value="6.5"/>
   <xacro:property name="joint_4_damping" value="0.01"/>
   <xacro:property name="joint_4_friction" value="3.48"/>
@@ -30,5 +30,5 @@
   <xacro:property name="joint_5_upper_limit" value="${pi}"/>
   <xacro:property name="joint_5_velocity_limit" value="6.283"/>
-  <xacro:property name="joint_5_torque_limit" value="6.8439285"/>
+  <xacro:property name="joint_5_torque_limit" value="6.5"/>
   <xacro:property name="joint_5_damping" value="0.01"/>
   <xacro:property name="joint_5_friction" value="3.48"/>
